Commit message: Add files via upload

File: urdf/DROK_P.urdf (robot description, URDF)
Before this commit: robot DROK_P, 22 links, 21 joints
Links:
- removed link ARM BASE
- removed link ARM1
- removed link ARM2
- removed link ARM3
- removed link ARM4
- removed link ARM5
- removed link BL
- removed link BLF
- removed link BR
- removed link BRF
- removed link FL
- removed link FLF
- removed link FR
- removed link FRF
- removed link L1
- removed link L2
- removed link L3
- removed link R1
- removed link R2
- removed link R3
- removed link sensor_frame
- added link arm_assembly; visual cylinder length=0.2 radius=0.05
- added link imu_link
- added link velodyne
- link base_link: mass 32.22 -> None; geometry visual box size=0.4 0.3 0.2
Joints:
- removed joint ARM BASE_JOINT
- removed joint ARM1_JOINT
- removed joint ARM2_JOINT
- removed joint ARM3_JOINT
- removed joint ARM4_JOINT
- removed joint ARM5_JOINT
- removed joint BLF_JOINT
- removed joint BL_JOINT
- removed joint BRF_JOINT
- removed joint BR_JOINT
- removed joint FLF_JOINT
- removed joint FL_JOINT
- removed joint FRF_JOINT
- removed joint FR_JOINT
- removed joint L1_JOINT
- removed joint L2_JOINT
- removed joint L3_JOINT
- removed joint R1_JOINT
- removed joint R2_JOINT
- removed joint R3_JOINT
- removed joint lidar_joint
- added joint arm_base_joint: type fixed, parent base_link, child arm_assembly, origin xyz=0.1 0 0 rpy=0 0 0
- added joint imu_joint: type fixed, parent base_link, child imu_link, origin xyz=0 0 0 rpy=0 0 0
- added joint velodyne_joint: type fixed, parent base_link, child velodyne, origin xyz=0.0 0.0 0.04 rpy=0 0 0
